File: hardware/usb_air_quality_sensor.sch (KiCad schematic (older format))
At the start: 14 parts

Commit message: bom
Parts:
- removed J?: USB_B_Micro, symbol Connector:USB_B_Micro
- removed R? (x2): 22, symbol Device:R
- removed U?: ATmega32U4-AU, Package_QFP:TQFP-44_10x10mm_P0.8mm, symbol MCU_Microchip_ATmega:ATmega32U4-AU
- added J?: USB_A, symbol Connector:USB_A
- added U?: ESP8266EX, Package_DFN_QFN:QFN-32-1EP_5x5mm_P0.5mm_EP3.45x3.45mm, symbol MCU_Espressif:ESP8266EX
Connections:
- wire segments 28 -> 20
Changed lines of the file:
@@
 $EndDescr
-$Comp
-L MCU_Microchip_ATmega:ATmega32U4-AU U?
-U 1 1 5E0AF899
-P 3800 3800
-F 0 "U?" H 3800 1911 50  0000 C CNN
-F 1 "ATmega32U4-AU" H 3800 1820 50  0000 C CNN
-F 2 "Package_QFP:TQFP-44_10x10mm_P0.8mm" H 3800 3800 50  0001 C CIN
-F 3 "http://ww1.microchip.com/downloads/en/DeviceDoc/Atmel-7766-8-bit-AVR-ATmega16U4-32U4_Datasheet.pdf" H 3800 3800 50  0001 C CNN
-	1    3800 3800
-	1    0    0    -1
-$EndComp
 $Comp
 L Sensor:BME280 U?
@@
 $EndComp
 $Comp
-L Connector:USB_B_Micro J?
-U 1 1 5E0B56D8
-P 2200 3300
-F 0 "J?" H 2257 3767 50  0000 C CNN
-F 1 "USB_B_Micro" H 2257 3676 50  0000 C CNN
-F 2 "" H 2350 3250 50  0001 C CNN
-F 3 "~" H 2350 3250 50  0001 C CNN
-	1    2200 3300
-	1    0    0    -1
-$EndComp
-$Comp
-L power:GND #PWR?
-U 1 1 5E0B61AE
-P 2100 3700
-F 0 "#PWR?" H 2100 3450 50  0001 C CNN
-F 1 "GND" H 2105 3527 50  0000 C CNN
-F 2 "" H 2100 3700 50  0001 C CNN
-F 3 "" H 2100 3700 50  0001 C CNN
-	1    2100 3700
-	1    0    0    -1
-$EndComp
-Wire Wire Line
-	2200 3700 2100 3700
-Connection ~ 2100 3700
-$Comp
-L Device:R R?
-U 1 1 5E0BAFBF
-P 2900 3400
-F 0 "R?" V 3000 3400 50  0000 C CNN
-F 1 "22" V 2900 3400 50  0000 C CNN
-F 2 "" V 2830 3400 50  0001 C CNN
-F 3 "~" H 2900 3400 50  0001 C CNN
-	1    2900 3400
-	0    1    1    0
-$EndComp
-Wire Wire Line
-	2500 3400 2750 3400
-Wire Wire Line
-	2750 3300 2500 3300
-$Comp
-L Device:R R?
-U 1 1 5E0BA8B6
-P 2900 3300
-F 0 "R?" V 2800 3300 50  0000 C CNN
-F 1 "22" V 2900 3300 50  0000 C CNN
-F 2 "" V 2830 3300 50  0001 C CNN
-F 3 "~" H 2900 3300 50  0001 C CNN
-	1    2900 3300
-	0    1    1    0
-$EndComp
-Wire Wire Line
-	3200 3300 3050 3300
-Wire Wire Line
-	3200 3400 3050 3400
-Wire Wire Line
-	2500 3100 2600 3100
-$Comp
-L power:+5V #PWR?
-U 1 1 5E0D56E1
-P 2600 2700
-F 0 "#PWR?" H 2600 2550 50  0001 C CNN
-F 1 "+5V" H 2615 2873 50  0000 C CNN
-F 2 "" H 2600 2700 50  0001 C CNN
-F 3 "" H 2600 2700 50  0001 C CNN
-	1    2600 2700
-	1    0    0    -1
-$EndComp
-Wire Wire Line
-	2600 3100 2600 2700
-Wire Wire Line
-	2600 3100 3200 3100
-Connection ~ 2600 3100
-$Comp
 L Regulator_Linear:XC6206PxxxMR U?
 U 1 1 5E0DA486
@@
 	1300 7150 1300 6850
 Connection ~ 1700 7150
-Text Label 2900 3100 0    50   ~ 0
-+5V
 Text Label 1300 6400 0    50   ~ 0
 +5V
@@
 	1    0    0    -1
 $EndComp
+$Comp
+L Connector:USB_A J?
+U 1 1 5E105FA6
+P 1800 2850
+F 0 "J?" H 1857 3317 50  0000 C CNN
+F 1 "USB_A" H 1857 3226 50  0000 C CNN
+F 2 "" H 1950 2800 50  0001 C CNN
+F 3 " ~" H 1950 2800 50  0001 C CNN
+	1    1800 2850
+	1    0    0    -1
+$EndComp
+$Comp
+L MCU_Espressif:ESP8266EX U?
+U 1 1 5E106CC0
+P 4050 2900
+F 0 "U?" H 4050 1711 50  0000 C CNN
+F 1 "ESP8266EX" H 4050 1620 50  0000 C CNN
+F 2 "Package_DFN_QFN:QFN-32-1EP_5x5mm_P0.5mm_EP3.45x3.45mm" H 4050 1600 50  0001 C CNN
+F 3 "http://espressif.com/sites/default/files/documentation/0a-esp8266ex_datasheet_en.pdf" H 4150 1600 50  0001 C CNN
+	1    4050 2900
+	1    0    0    -1
+$EndComp

Commit message: wip
Parts:
- removed U?: BME280, Package_LGA:Bosch_LGA-8_2.5x2.5mm_P0.65mm_ClockwisePinNumbering, symbol Sensor:BME280
- added C?: 0.1 uF, symbol Device:C_Small
- added R?: 12K, symbol Device:R
- added R? (x2): 27, symbol Device:R_Small
- added R?: 1.5K, symbol Device:R_Small
- added U?: HDC1080, Package_SON:Texas_PWSON-N6, symbol Sensor_Humidity:HDC1080
- added U?: FT232RL, Package_SO:SSOP-28_5.3x10.2mm_P0.65mm, symbol Interface_USB:FT232RL
- added U?: PL2303SA, Package_SO:SO-8_3.9x4.9mm_P1.27mm, symbol lib:PL2303SA
- added U?: W25Q32JVSS, Package_SO:SOIC-8_5.23x5.23mm_P1.27mm, symbol Memory_Flash:W25Q32JVSS
- added Y?: Crystal, symbol Device:Crystal
Connections:
- net labels added: PL_RXD, PL_TXD
- wire segments 20 -> 41
- no-connect marks 0 -> 1
Other:
- moved on the sheet: J?

Commit message: wip
Parts:
- removed Y?: Crystal, symbol Device:Crystal
- added C? (x2): 22 pF, symbol Device:C_Small
- added R?: 499, symbol Device:R_Small
- added XTAL?: 26 MHz, symbol Device:Crystal_GND24
Connections:
- net +3V3: now also U?.8 (VCC)
- net GND: now also U?.4 (GND), C?.1, C?.2, XTAL?.2, XTAL?.4
- net PL_RXD: now also R?.1; no longer U?.26 (U0TXD)
- net SDIO_2: now reaches U?.18 (SDIO_DATA_2)
- net SDIO_2: now also U?.3 (IO2)
- net SDIO_3: now reaches U?.19 (SDIO_DATA_3)
- net SDIO_3: now also U?.7 (IO3)
- net SDCS: now reaches U?.20 (SDIO_CMD)
- net SDCS: now also U?.1 (~CS)
- net SDCLK: now reaches U?.21 (SDIO_CLK)
- net SDCLK: now also U?.6 (CLK)
- net SDIO_0: now reaches U?.22 (SDIO_DATA_0)
- net SDIO_0: now also U?.5 (DI(IO0))
- net SDIO_1: now reaches U?.23 (SDIO_DATA_1)
- net SDIO_1: now also U?.2 (DO(IO1))
- net at U?.27 (XTAL_OUT): now also C?.1, XTAL?.3
- net at U?.28 (XTAL_IN): now also C?.2, XTAL?.1
- new net: R?.2, U?.26 (U0TXD)
Other:
- moved on the sheet: C?, J?, R?, U?

Commit message: wip
Parts:
- removed C? (x2): 100 nF, symbol Device:C
- removed R? (x2): 2K, symbol Device:R
- removed U?: FT232RL, Package_SO:SSOP-28_5.3x10.2mm_P0.65mm, symbol Interface_USB:FT232RL
- added C8: 0.1 uF, symbol Device:C_Small
- added R6, R7: 1k, symbol Device:R_Small
- gave numbers to parts that had none: 19
Connections:
- net +3V3: now also U5.5 (VCC), C8.1, R6.1, R7.1
- net GND: now also U3.33 (GND), U5.2 (GND), C8.2
- net SDIO_0: now also U1.2 (DO(IO1)), U3.15 (GPIO0)
- net SDA: now reaches U3.14 (GPIO2)
- net SDA: now also U5.1 (SDA), R6.2
- net SCL: now reaches U3.9 (MTMS)
- net SCL: now also U5.6 (SCL), R7.2
- net SDIO_1: no longer names the net of U3.23 (SDIO_DATA_1)
- net SDIO_1: no longer U1.2 (DO(IO1))
Other:
- moved on the sheet: R2, U1, U5
