File: hardware/usb_air_quality_sensor.sch (KiCad schematic (older format))
At the start: 36 parts, among them J1 USB_A, U1 W25Q32JVSS, U3 ESP8266EX, U4 PL2303SA, U5 HDC1080

Commit message: one percent
Parts:
- R?: value 12K -> 12K;1%
Changed lines of the file:
@@
 U 1 1 5E2E9A46
 P 2750 4250
-F 0 "R?" V 2650 4100 50  0000 C CNN
-F 1 "12K" V 2650 4250 50  0000 C CNN
+F 0 "R?" V 2700 4050 50  0000 C CNN
+F 1 "12K;1%" V 2650 4250 50  0000 C CNN
 F 2 "" H 2750 4250 50  0001 C CNN
 F 3 "~" H 2750 4250 50  0001 C CNN

Commit message: netlist
Parts:
- gave numbers to parts that had none: 16
- renumbered C5 to C12, C6 to C14, C8 to C15, C7 to C16, C1 to C3, C3 to C5, C4 to C8, R2 to R4, R6 to R5, R7 to R6, R3 to R7, R4 to R8, R5 to R9, U3 to U2, U1 to U3, U5 to U4, U4 to U5

Commit message: power led
Parts:
- added D?: PWR LED, symbol Device:LED_Small
- added R?: 220, symbol Device:R_Small
Connections:
- net +3V3: now also R?.1
- net GND: now also D?.1 (K)
- new net: D?.2 (A), R?.2
Changed lines of the file:
@@
 Wire Wire Line
 	7350 2550 7350 3650
+$Comp
+L power:+3.3V #PWR?
+U 1 1 5E4BC0C0
+P 4100 6400
+F 0 "#PWR?" H 4100 6250 50  0001 C CNN
+F 1 "+3.3V" H 4115 6573 50  0000 C CNN
+F 2 "" H 4100 6400 50  0001 C CNN
+F 3 "" H 4100 6400 50  0001 C CNN
+	1    4100 6400
+	1    0    0    -1
+$EndComp
+$Comp
+L Device:R_Small R?
+U 1 1 5E4BD4BB
+P 4100 6600
+F 0 "R?" H 4159 6646 50  0000 L CNN
+F 1 "220" H 4159 6555 50  0000 L CNN
+F 2 "" H 4100 6600 50  0001 C CNN
+F 3 "~" H 4100 6600 50  0001 C CNN
+	1    4100 6600
+	1    0    0    -1
+$EndComp
+Wire Wire Line
+	4100 6400 4100 6500
+$Comp
+L Device:LED_Small D?
+U 1 1 5E4C4B2D
+P 4100 6850
+F 0 "D?" V 4146 6948 50  0000 L CNN
+F 1 "PWR LED" V 4055 6948 50  0000 L CNN
+F 2 "" V 4100 6850 50  0001 C CNN
+F 3 "~" V 4100 6850 50  0001 C CNN
+	1    4100 6850
+	0    1    -1   0
+$EndComp
+$Comp
+L power:GND #PWR?
+U 1 1 5E4C5946
+P 4100 7000
+F 0 "#PWR?" H 4100 6750 50  0001 C CNN
+F 1 "GND" H 4105 6827 50  0000 C CNN
+F 2 "" H 4100 7000 50  0001 C CNN
+F 3 "" H 4100 7000 50  0001 C CNN
+	1    4100 7000
+	1    0    0    -1
+$EndComp
+Wire Wire Line
+	4100 6950 4100 7000
+Wire Wire Line
+	4100 6750 4100 6700
 $EndSCHEMATC

Commit message: netlist
Parts:
- gave numbers to parts that had none: 2
Changed lines of the file:
@@
 	7350 2550 7350 3650
 $Comp
-L power:+3.3V #PWR?
+L power:+3.3V #PWR0101
 U 1 1 5E4BC0C0
 P 4100 6400
-F 0 "#PWR?" H 4100 6250 50  0001 C CNN
+F 0 "#PWR0101" H 4100 6250 50  0001 C CNN
 F 1 "+3.3V" H 4115 6573 50  0000 C CNN
 F 2 "" H 4100 6400 50  0001 C CNN
@@
 $EndComp
 $Comp
-L Device:R_Small R?
+L Device:R_Small R10
 U 1 1 5E4BD4BB
 P 4100 6600
-F 0 "R?" H 4159 6646 50  0000 L CNN
+F 0 "R10" H 4159 6646 50  0000 L CNN
 F 1 "220" H 4159 6555 50  0000 L CNN
 F 2 "" H 4100 6600 50  0001 C CNN
@@
 	4100 6400 4100 6500
 $Comp
-L Device:LED_Small D?
+L Device:LED_Small D1
 U 1 1 5E4C4B2D
 P 4100 6850
-F 0 "D?" V 4146 6948 50  0000 L CNN
+F 0 "D1" V 4146 6948 50  0000 L CNN
 F 1 "PWR LED" V 4055 6948 50  0000 L CNN
 F 2 "" V 4100 6850 50  0001 C CNN
@@
 $EndComp
 $Comp
-L power:GND #PWR?
+L power:GND #PWR0102
 U 1 1 5E4C5946
 P 4100 7000
-F 0 "#PWR?" H 4100 6750 50  0001 C CNN
+F 0 "#PWR0102" H 4100 6750 50  0001 C CNN
 F 1 "GND" H 4105 6827 50  0000 C CNN
 F 2 "" H 4100 7000 50  0001 C CNN
