File: hardware/usb_air_quality_sensor.sch (KiCad schematic (older format))
At the start: 38 parts, among them J1 USB_A, SW1 SW_Push_45deg, U1 AP1117-33, U2 ESP8266EX, U3 W25Q32JVSS, U4 HDC1080, U5 PL2303SA

Commit message: wip
Connections:
- net +3V3: now also C15.1, R5.1, R6.1, U4.5 (VCC)
Other:
- moved on the sheet: C15
Changed lines of the file:
@@
 P 9600 4200
 F 0 "R8" V 9700 4200 50  0000 C CNN
-F 1 "27" V 9600 4200 50  0000 C CNN
+F 1 "27" V 9550 4350 50  0000 C CNN
 F 2 "" H 9600 4200 50  0001 C CNN
 F 3 "~" H 9600 4200 50  0001 C CNN
@@
 P 9600 4100
 F 0 "R7" V 9500 4100 50  0000 C CNN
-F 1 "27" V 9600 4100 50  0000 C CNN
+F 1 "27" V 9550 4250 50  0000 C CNN
 F 2 "" H 9600 4100 50  0001 C CNN
 F 3 "~" H 9600 4100 50  0001 C CNN
@@
 L Device:C_Small C15
 U 1 1 5E20FAD2
-P 7650 5100
-F 0 "C15" H 7742 5146 50  0000 L CNN
-F 1 "0.1 uF" H 7742 5055 50  0000 L CNN
-F 2 "" H 7650 5100 50  0001 C CNN
-F 3 "~" H 7650 5100 50  0001 C CNN
-	1    7650 5100
+P 7450 5100
+F 0 "C15" H 7542 5146 50  0000 L CNN
+F 1 "0.1 uF" H 7542 5055 50  0000 L CNN
+F 2 "" H 7450 5100 50  0001 C CNN
+F 3 "~" H 7450 5100 50  0001 C CNN
+	1    7450 5100
 	1    0    0    -1
 $EndComp
@@
 L power:+3.3V #PWR023
 U 1 1 5E218028
-P 7650 4600
-F 0 "#PWR023" H 7650 4450 50  0001 C CNN
-F 1 "+3.3V" H 7665 4773 50  0000 C CNN
-F 2 "" H 7650 4600 50  0001 C CNN
-F 3 "" H 7650 4600 50  0001 C CNN
-	1    7650 4600
-	1    0    0    -1
-$EndComp
-Wire Wire Line
-	7650 4650 7650 5000
+P 7350 4650
+F 0 "#PWR023" H 7350 4500 50  0001 C CNN
+F 1 "+3.3V" H 7500 4700 50  0000 C CNN
+F 2 "" H 7350 4650 50  0001 C CNN
+F 3 "" H 7350 4650 50  0001 C CNN
+	1    7350 4650
+	1    0    0    -1
+$EndComp
+Wire Wire Line
+	7450 4650 7450 5000
 Connection ~ 6700 5500
 Wire Wire Line
@@
 $EndComp
 Wire Wire Line
-	6700 4650 7650 4650
+	6700 4650 7350 4650
 Wire Wire Line
 	6700 4650 6250 4650
@@
 	7350 4000 7350 4350
 Wire Wire Line
-	7650 5200 7650 5500
-Wire Wire Line
-	6700 5500 7650 5500
+	7450 5200 7450 5500
+Wire Wire Line
+	6700 5500 7450 5500
 Wire Wire Line
 	8100 4200 7400 4200
@@
 Wire Wire Line
 	4100 6900 4100 6800
+Connection ~ 7350 4650
+Wire Wire Line
+	7350 4650 7450 4650
 $EndSCHEMATC

Commit message: wip
Changed lines of the file:
@@
 L power:+3.3V #PWR028
 U 1 1 5E1723AE
-P 10150 3550
-F 0 "#PWR028" H 10150 3400 50  0001 C CNN
-F 1 "+3.3V" H 10165 3723 50  0000 C CNN
-F 2 "" H 10150 3550 50  0001 C CNN
-F 3 "" H 10150 3550 50  0001 C CNN
-	1    10150 3550
+P 9950 3550
+F 0 "#PWR028" H 9950 3400 50  0001 C CNN
+F 1 "+3.3V" H 9965 3723 50  0000 C CNN
+F 2 "" H 9950 3550 50  0001 C CNN
+F 3 "" H 9950 3550 50  0001 C CNN
+	1    9950 3550
 	1    0    0    -1
 $EndComp
@@
 Connection ~ 9950 3550
 Wire Wire Line
-	9950 3550 10150 3550
-Wire Wire Line
 	10000 4100 9950 4100

Commit message: pcb
Parts:
- removed C2, C8: 6.8 pF, symbol Device:C_Small
- removed XTAL1: 26 MHz, symbol Device:Crystal_GND24
- added C? (x2): C_Small, symbol Device:C_Small
- added D?: TX LED, symbol Device:LED_Small
- added R?: 470, symbol Device:R_Small
- added Y?: Crystal_Small, symbol Device:Crystal_Small
- R10: value 220 -> 470
Connections:
- net +3V3: now also R?.1
- net GND: now also C?.2, C?.2
- net at R4.2, U2.26 (U0TXD): now also D?.1 (K)
- net at U2.27 (XTAL_OUT): now also C?.1, Y?.1
- net at U2.28 (XTAL_IN): now also C?.1, Y?.2
- new net: D?.2 (A), R?.2
Other:
- moved on the sheet: R3
Changed lines of the file:
@@
-$EndComp
-$Comp
-L Device:Crystal_GND24 XTAL1
-U 1 1 5E1A84F0
-P 2100 5100
-F 0 "XTAL1" V 2300 5450 50  0000 R CNN
-F 1 "26 MHz" V 2200 5550 50  0000 R CNN
-F 2 "" H 2100 5100 50  0001 C CNN
-F 3 "~" H 2100 5100 50  0001 C CNN
-	1    2100 5100
-	0    -1   -1   0
 $EndComp
 $Comp
@@
 	1    0    0    -1
 $EndComp
-Wire Wire Line
-	2100 5250 2100 5350
-Wire Wire Line
-	2100 5350 2350 5350
-Wire Wire Line
-	2100 4950 2100 4850
-Wire Wire Line
-	2100 4850 2950 4850
-$Comp
-L power:GND #PWR03
-U 1 1 5E1FA286
-P 1850 5350
-F 0 "#PWR03" H 1850 5100 50  0001 C CNN
-F 1 "GND" H 1855 5177 50  0000 C CNN
-F 2 "" H 1850 5350 50  0001 C CNN
-F 3 "" H 1850 5350 50  0001 C CNN
-	1    1850 5350
-	1    0    0    -1
-$EndComp
-Wire Wire Line
-	1900 5100 1850 5100
-Wire Wire Line
-	1850 5100 1850 5350
-$Comp
-L power:GND #PWR011
-U 1 1 5E1FB8E3
-P 2450 5100
-F 0 "#PWR011" H 2450 4850 50  0001 C CNN
-F 1 "GND" V 2455 4972 50  0000 R CNN
-F 2 "" H 2450 5100 50  0001 C CNN
-F 3 "" H 2450 5100 50  0001 C CNN
-	1    2450 5100
-	0    -1   -1   0
-$EndComp
-Wire Wire Line
-	2300 5100 2350 5100
-$Comp
-L Device:C_Small C8
-U 1 1 5E2042AB
-P 2350 5250
-F 0 "C8" H 2442 5296 50  0000 L CNN
-F 1 "6.8 pF" H 2442 5205 50  0000 L CNN
-F 2 "" H 2350 5250 50  0001 C CNN
-F 3 "~" H 2350 5250 50  0001 C CNN
-	1    2350 5250
-	1    0    0    -1
-$EndComp
-Connection ~ 2350 5350
-Wire Wire Line
-	2350 5350 2950 5350
-Wire Wire Line
-	2350 5150 2350 5100
-Connection ~ 2350 5100
-Wire Wire Line
-	2350 5100 2450 5100
-$Comp
-L Device:C_Small C2
-U 1 1 5E2054F0
-P 1500 5050
-F 0 "C2" H 1300 5050 50  0000 L CNN
-F 1 "6.8 pF" H 1250 4950 50  0000 L CNN
-F 2 "" H 1500 5050 50  0001 C CNN
-F 3 "~" H 1500 5050 50  0001 C CNN
-	1    1500 5050
-	1    0    0    -1
-$EndComp
-Wire Wire Line
-	1500 5150 1500 5350
-Wire Wire Line
-	1500 5350 1850 5350
-Connection ~ 1850 5350
-Wire Wire Line
-	1500 4950 1500 4850
-Wire Wire Line
-	1500 4850 2100 4850
-Connection ~ 2100 4850
 $Comp
 L power:+3.3V #PWR020
@@
 	4750 4050 5300 4050
 Wire Wire Line
-	5300 4050 5300 3550
-Wire Wire Line
 	5300 3550 6100 3550
 Wire Wire Line
@@
 Wire Wire Line
 	5250 3650 6100 3650
-Wire Wire Line
-	4750 4450 5450 4450
 Wire Wire Line
 	4750 4350 7350 4350
@@
 L Device:R_Small R3
 U 1 1 5E3F4D43
-P 5000 3350
-F 0 "R3" H 5059 3396 50  0000 L CNN
-F 1 "200" H 5059 3305 50  0000 L CNN
-F 2 "" H 5000 3350 50  0001 C CNN
-F 3 "~" H 5000 3350 50  0001 C CNN
-	1    5000 3350
+P 5000 2800
+F 0 "R3" H 5059 2846 50  0000 L CNN
+F 1 "200" H 5059 2755 50  0000 L CNN
+F 2 "" H 5000 2800 50  0001 C CNN
+F 3 "~" H 5000 2800 50  0001 C CNN
+	1    5000 2800
 	1    0    0    -1
 $EndComp
@@
 NoConn ~ 2950 4450
 Wire Wire Line
-	5000 3950 5000 3450
+	5000 3950 5000 2900
 Wire Wire Line
 	4750 3950 5000 3950
@@
 	4750 3850 4950 3850
 Wire Wire Line
-	5000 3250 5000 2550
+	5000 2700 5000 2550
 Wire Wire Line
 	5000 2550 7350 2550
@@
 P 4100 6700
 F 0 "R10" H 4159 6746 50  0000 L CNN
-F 1 "220" H 4159 6655 50  0000 L CNN
+F 1 "470" H 4159 6655 50  0000 L CNN
 F 2 "" H 4100 6700 50  0001 C CNN
 F 3 "~" H 4100 6700 50  0001 C CNN
@@
 Wire Wire Line
 	7350 4650 7450 4650
+$Comp
+L power:+3.3V #PWR?
+U 1 1 5E15541A
+P 5150 3250
+F 0 "#PWR?" H 5150 3100 50  0001 C CNN
+F 1 "+3.3V" H 5165 3423 50  0000 C CNN
+F 2 "" H 5150 3250 50  0001 C CNN
+F 3 "" H 5150 3250 50  0001 C CNN
+	1    5150 3250
+	1    0    0    -1
+$EndComp
+$Comp
+L Device:LED_Small D?
+U 1 1 5E155427
+P 5150 3750
+F 0 "D?" V 5196 3848 50  0000 L CNN
+F 1 "TX LED" V 5105 3848 50  0000 L CNN
+F 2 "" V 5150 3750 50  0001 C CNN
+F 3 "~" V 5150 3750 50  0001 C CNN
+	1    5150 3750
+	0    1    -1   0
+$EndComp
+Wire Wire Line
+	5300 3550 5300 4050
+Wire Wire Line
+	5150 3250 5150 3350
+Wire Wire Line
+	4750 4450 5150 4450
+Wire Wire Line
+	5150 3850 5150 4450
+Connection ~ 5150 4450
+Wire Wire Line
+	5150 4450 5450 4450
+Wire Wire Line
+	5150 3550 5150 3650
+$Comp
+L Device:R_Small R?
+U 1 1 5E155420
+P 5150 3450
+F 0 "R?" H 5209 3496 50  0000 L CNN
+F 1 "470" H 5209 3405 50  0000 L CNN
+F 2 "" H 5150 3450 50  0001 C CNN
+F 3 "~" H 5150 3450 50  0001 C CNN
+	1    5150 3450
+	1    0    0    -1
+$EndComp
+$Comp
+L Device:Crystal_Small Y?
+U 1 1 5E217484
+P 2300 5100
+F 0 "Y?" V 2254 5188 50  0000 L CNN
+F 1 "Crystal_Small" V 2345 5188 50  0000 L CNN
+F 2 "" H 2300 5100 50  0001 C CNN
+F 3 "~" H 2300 5100 50  0001 C CNN
+	1    2300 5100
+	0    1    1    0
+$EndComp
+Wire Wire Line
+	2300 5000 2300 4850
+Wire Wire Line
+	2300 4850 2950 4850
+Wire Wire Line
+	2300 5200 2300 5350
+Wire Wire Line
+	2300 5350 2950 5350
+$Comp
+L Device:C_Small C?
+U 1 1 5E24C193
+P 2050 4850
+F 0 "C?" V 1950 4750 50  0000 C CNN
+F 1 "C_Small" V 2000 4650 50  0000 C CNN
+F 2 "" H 2050 4850 50  0001 C CNN
+F 3 "~" H 2050 4850 50  0001 C CNN
+	1    2050 4850
+	0    1    1    0
+$EndComp
+Wire Wire Line
+	2150 4850 2300 4850
+Connection ~ 2300 4850
+$Comp
+L Device:C_Small C?
+U 1 1 5E2541A8
+P 2050 5350
+F 0 "C?" V 2100 5250 50  0000 C CNN
+F 1 "C_Small" V 2200 5150 50  0000 C CNN
+F 2 "" H 2050 5350 50  0001 C CNN
+F 3 "~" H 2050 5350 50  0001 C CNN
+	1    2050 5350
+	0    1    1    0
+$EndComp
+Wire Wire Line
+	2150 5350 2300 5350
+Connection ~ 2300 5350
+$Comp
+L power:GND #PWR?
+U 1 1 5E25B53C
+P 1850 5050
+F 0 "#PWR?" H 1850 4800 50  0001 C CNN
+F 1 "GND" V 1855 4922 50  0000 R CNN
+F 2 "" H 1850 5050 50  0001 C CNN
+F 3 "" H 1850 5050 50  0001 C CNN
+	1    1850 5050
+	0    1    1    0
+$EndComp
+Wire Wire Line
+	1850 4850 1850 5050
+Wire Wire Line
+	1850 5050 1850 5350
+Connection ~ 1850 5050
+Wire Wire Line
+	1850 5350 1950 5350
+Wire Wire Line
+	1850 4850 1950 4850
 $EndSCHEMATC
